Commit message: Begin orange pixel detection and motor control

File: csc790_labs/src/lab03/lab03_description/urdf/lab03.gazebo.xacro (robot description, xacro)
@@ -1,79 +1,80 @@
 <?xml version="1.0"?>
 <robot xmlns:xacro="http://www.ros.org/wiki/xacro" name="lab03">
-	<gazebo>
-		<plugin name="gazebo_ros_control" filename="libgazebo_ros_control.so">
-			<robotNamespace>/lab03</robotNamespace>
-		</plugin>
-	</gazebo>
-	<gazebo reference="robot chassis">
-		<material>Gazebo/Blue</material>
-	</gazebo>
-	<gazebo reference="left_wheel">
-		<material>Gazebo/Black</material>
-	</gazebo>
-	<gazebo reference="right_wheel">
-		<material>Gazebo/Black</material>
-	</gazebo>
-	<gazebo reference="front_glide">
-		<material>Gazebo/Blue</material>
-	</gazebo>
-	<gazebo reference="back_glide">
-		<material>Gazebo/Blue</material>
-	</gazebo>
-	<!-- camera -->
-  <gazebo reference="camera_link">
-    <sensor type="camera" name="camera1">
-      <update_rate>10.0</update_rate>
-      <camera name="head">
-        <horizontal_fov>1.3962634</horizontal_fov>
-        <image>
-          <width>800</width>
-          <height>800</height>
-          <format>R8G8B8</format>
-        </image>
-        <clip>
-          <near>0.02</near>
-          <far>300</far>
-        </clip>
-        <noise>
-          <type>gaussian</type>
-          <!-- Noise is sampled independently per pixel on each frame.
-               That pixel's noise value is added to each of its color
-               channels, which at that point lie in the range [0,1]. -->
-          <mean>0.0</mean>
-          <stddev>0.007</stddev>
-        </noise>
-      </camera>
-      <plugin name="camera_controller" filename="libgazebo_ros_camera.so">
-        <alwaysOn>true</alwaysOn>
-        <updateRate>0.0</updateRate>
-        <cameraName>lab03/camera1</cameraName>
-        <imageTopicName>image_raw</imageTopicName>
-        <cameraInfoTopicName>camera_info</cameraInfoTopicName>
-        <frameName>camera_link</frameName>
-        <hackBaseline>0.07</hackBaseline>
-        <distortionK1>0.0</distortionK1>
-        <distortionK2>0.0</distortionK2>
-        <distortionK3>0.0</distortionK3>
-        <distortionT1>0.0</distortionT1>
-        <distortionT2>0.0</distortionT2>
-      </plugin>
-    </sensor>
-  </gazebo>
-  <gazebo>
-  	<plugin name="differential_drive_controller" filename="libgazebo_ros_diff_drive.so">
-  		<alwaysOn>true</alwaysOn>
-  		<updateRate>10</updateRate>
-  		<leftJoint>left_wheel_joint</leftJoint>
-  		<rightJoint>right_wheel_joint</rightJoint>
-  		<wheelSeperation>${(ch_radius * wh_radius) * 2}</wheelSeperation>
-  		<wheelDiameter>${wh_radius * 2}</wheelDiameter>
-  		<torque>20</torque>
-  		<commandTopic>cmd_vel</commandTopic>
-  		<odometryTopic>odom</odometryTopic>
-  		<odometryFrame>odom</odometryFrame>
-  		<robotBaseFrame>robot_chassis</robotBaseFrame>
-  		<legacyMode>false</legacyMode>
-  	</plugin>
-  </gazebo>
+    <gazebo reference="robot_chassis">
+        <material>Gazebo/DarkGray</material>
+    </gazebo>
+    <gazebo reference="left_wheel">
+        <material>Gazebo/White</material>
+    </gazebo>
+    <gazebo reference="right_wheel">
+        <material>Gazebo/White</material>
+    </gazebo>
+    <gazebo reference="front_glide">
+        <material>Gazebo/Blue</material>
+    </gazebo>
+    <gazebo reference="rear_glide">
+        <material>Gazebo/Blue</material>
+    </gazebo>
+    <gazebo reference="camera">
+        <material>Gazebo/Red</material>
+    </gazebo>
+    <!-- Camera Plugin -->
+    <xacro:property name="camera_update_hz" value="10" />
+    <gazebo reference="camera">
+        <sensor type="camera" name="camera1">
+            <update_rate>${camera_update_hz}</update_rate>
+            <camera name="head">
+                <horizontal_fov>1.3962634</horizontal_fov>
+                <image>
+                    <width>640</width>
+                    <height>480</height>
+                    <format>R8G8B8</format>
+                </image>
+                <clip>
+                    <near>0.02</near>
+                    <far>300</far>
+                </clip>
+                <noise>
+                    <type>gaussian</type>
+                    <mean>0.0</mean>
+                    <stddev>0.007</stddev>
+                </noise>
+            </camera>
+            <plugin name="camera_controller" filename="libgazebo_ros_camera.so">
+                <alwaysOn>true</alwaysOn>
+                <updateRate>0.0</updateRate>
+                <cameraName>lab03/camera1</cameraName>
+                <imageTopicName>image_raw</imageTopicName>
+                <cameraInfoTopicName>camera_info</cameraInfoTopicName>
+                <frameName>camera</frameName>
+                <hackBaseline>0.07</hackBaseline>
+                <distortionK1>0.0</distortionK1>
+                <distortionK2>0.0</distortionK2>
+                <distortionK3>0.0</distortionK3>
+                <distortionT1>0.0</distortionT1>
+                <distortionT2>0.0</distortionT2>
+            </plugin>
+        </sensor>
+    </gazebo>
+    <!-- Differential Drive Plugin -->
+    <xacro:property name="diffdrive_update_hz" value="10" />
+    <!-- TODO:
+            parameterize elements below
+     -->
+    <gazebo>
+        <plugin name="differential_drive_controller" filename="libgazebo_ros_diff_drive.so">
+            <alwaysOn>true</alwaysOn>
+            <updateRate>${diffdrive_update_hz}</updateRate>
+            <leftJoint>left_wheel_joint</leftJoint>
+            <rightJoint>right_wheel_joint</rightJoint>
+            <wheelSeparation>${(chassis_radius - wheel_radius) * 2}</wheelSeparation>
+            <wheelDiameter>${wheel_radius * 2}</wheelDiameter>
+            <torque>20</torque>
+            <commandTopic>cmd_vel</commandTopic>
+            <odometryTopic>odom</odometryTopic>
+            <odometryFrame>odom</odometryFrame>
+            <robotBaseFrame>robot_chassis</robotBaseFrame>
+            <legacyMode>false</legacyMode>
+        </plugin>
+    </gazebo>
 </robot>

File: csc790_labs/src/lab03/lab03_description/urdf/lab03.macros.xacro (robot description, xacro)
@@ -1,78 +1,113 @@
 <?xml version="1.0"?>
 <robot xmlns:xacro="http://www.ros.org/wiki/xacro" name="lab03">
-	  <xacro:macro name="wheel" params="reflect_lr suffix">
+    <!-- Create cylinder geometry -->
+    <xacro:macro name="create_cylinder_geometry" params="radius length">
+        <origin xyz="0 0 0" rpy="0 0 0" />
+        <geometry>
+            <cylinder radius="${radius}" length="${length}" />
+        </geometry>
+    </xacro:macro>
+    <!-- Create sphere geometry -->
+    <xacro:macro name="create_sphere_geometry" params="radius">
+        <origin xyz="0 0 0" rpy="0 0 0" />
+        <geometry>
+            <sphere radius="${radius}" />
+        </geometry>
+    </xacro:macro>
+    <!-- Macro for creating a cylinder inertial element -->
+    <xacro:macro name="create_cylinder_inertial" params="mass radius length">
+        <inertial>
+            <mass value="${mass}" />
+            <origin xyz="0 0 0" rpy="0 0 0" />
+            <inertia
+                ixx="${(1/12)*mass*(3*radius**2 + length**2)}"
+                ixy="0"
+                ixz="0"
+                iyy="${(1/12)*mass*(3*radius**2 + length**2)}"
+                iyz="0"
+                izz="${(1/2)*mass*radius**2}"
+                />
+        </inertial>
+    </xacro:macro>
+    <!-- Macro for creating a sphere inertial element -->
+    <xacro:macro name="create_sphere_inertial" params="mass radius">
+        <inertial>
+            <mass value="${mass}" />
+            <inertia
+                ixx="${(2/5) * mass * radius * radius}"
+                ixy="0"
+                ixz="0"
+                iyy="${(2/5) * mass * radius * radius}"
+                iyz="0"
+                izz="${(2/5) * mass * radius * radius}"
+                />
+        </inertial>
+    </xacro:macro>
+    <!--
+         Macro for creating wheels
+            reflect_lr  : left (1) or right (-1) wheel
+            wheel_id    : give the wheel a unique identifier
+            parent_name : the name of the wheel's parent
+    -->
+    <xacro:macro name="create_wheel" params="reflect_lr wheel_id parent_name">
         <!-- The name of the current wheel -->
-        <xacro:property name="wheel_name" value="${suffix}_wheel" />
-        <!-- Create the wheel geometry (for visual debug and collisions) -->
-        <xacro:property name="wheel_geometry">
-            <origin xyz="0 0 0" rpy="${PI/2} 0 0" />
-            <geometry>
-                <sphere radius="${wh_radius}" />
-            </geometry>
-        </xacro:property>
-         <link name="${wheel_name}">
+        <xacro:property name="wheel_name" value="${wheel_id}_wheel" />
+        <!-- The wheel's rigid body -->
+        <link name="${wheel_name}">
+            <!-- Create the wheel visual -->
             <visual>
-                <xacro:insert_block name="wheel_geometry" />
-                <material name="black" />
+                <xacro:create_sphere_geometry radius="${wheel_radius}" />
+                <material name="red" />
             </visual>
+            <!-- The wheel's collision shape -->
             <collision>
-                <xacro:insert_block name="wheel_geometry" />
+                <xacro:create_sphere_geometry radius="${wheel_radius}" />
             </collision>
-            <inertial>
-                <mass value="${wh_mass}" />
-                <origin xyz="0 0 0" rpy="${PI/2} 0 0" />
-                <inertia
-                    ixx="${(1/12)*wh_mass*(3*wh_radius**2 + wh_length**2)}"
-                    ixy="0"
-                    ixz="0"
-                    iyy="${(1/12)*wh_mass*(3*wh_radius**2 + wh_length**2)}"
-                    iyz="0"
-                    izz="${(1/2)*wh_mass*wh_radius**2}"
-                    />
-            </inertial>
+            <!-- Create the wheel's inertial matrix -->
+            <xacro:create_cylinder_inertial
+                mass="${wheel_mass}" radius="${wheel_radius}"
+                length="${wheel_length}"/>
         </link>
+        <!-- Connect the wheel to its parent -->
         <joint name="${wheel_name}_joint" type="continuous">
-            <parent link="robot_chassis" />
+            <parent link="${parent_name}" />
             <child link="${wheel_name}" />
-            <origin xyz = "${(ch_radius - wh_radius)*reflect_lr} 0 0" />
+            <origin xyz="0 ${(chassis_radius - wheel_radius * 1.1) * reflect_lr} 0" rpy="0 0 0" />
             <axis xyz="0 1 0" />
+            <!-- <limit effort="10" velocity="10" /> -->
         </joint>
     </xacro:macro>
-    <xacro:macro name="glide" params="reflect_lr suffix">
-        <!-- The name of the current wheel -->
-        <xacro:property name="glide_name" value="${suffix}_glide" />
-        <!-- Create the wheel geometry (for visual debug and collisions) -->
-        <xacro:property name="glide_geometry">
-            <origin xyz="0 0 0" rpy="${PI/2} 0 0" />
-            <geometry>
-                <sphere radius="${gl_radius}" />
-            </geometry>
-        </xacro:property>
-         <link name="${glide_name}">
+    <!--
+         Macro for creating glides
+            reflect_fr  : front (1) or rear (-1) glide
+            glide_id    : give the glide a unique identifier
+            parent_name : the name of the glide's parent
+    -->
+    <xacro:macro name="create_glide" params="reflect_fr glide_id parent_name">
+        <!-- The name of the current glide -->
+        <xacro:property name="glide_name" value="${glide_id}_glide" />
+        <!-- The glide's rigid body -->
+        <link name="${glide_name}">
+            <!-- Create the glide visual -->
             <visual>
-                <xacro:insert_block name="glide_geometry" />
-                <material name="white" />
+                <xacro:create_sphere_geometry radius="${glide_radius}" />
+                <material name="blue" />
             </visual>
+            <!-- The glide's collision shape -->
             <collision>
-                <xacro:insert_block name="glide_geometry" />
+                <xacro:create_sphere_geometry radius="${glide_radius}" />
             </collision>
-            <inertial>
-                <mass value="${gl_mass}" />
-                <origin xyz="0 0 0" rpy="${PI/2} 0 0" />
-                <inertia
-                    ixx="${(1/12)*gl_mass*(3*gl_radius**2 + wh_length**2)}"
-                    ixy="0"
-                    ixz="0"
-                    iyy="${(1/12)*gl_mass*(3*gl_radius**2 + wh_length**2)}"
-                    iyz="0"
-                    izz="${(1/2)*gl_mass*gl_radius**2}"
-                    />
-            </inertial>
+            <!-- Create the glide's inertial matrix -->
+            <xacro:create_sphere_inertial
+                mass="${glide_mass}" radius="${glide_radius}" />
         </link>
+        <!-- Connect the glide to its parent -->
         <joint name="${glide_name}_joint" type="fixed">
-            <parent link="robot_chassis" />
+            <parent link="${parent_name}" />
             <child link="${glide_name}" />
-            <origin xyz = "0 ${(ch_radius - gl_radius)*reflect_lr} 0" />
-            <axis xyz="0 1 0" />
+            <origin
+                xyz="${(chassis_radius - glide_radius) * reflect_fr} 0 ${-chassis_height/2}"
+                rpy="0 0 0" />
+            <!-- <limit effort="10" velocity="10" /> -->
         </joint>
     </xacro:macro>

File: csc790_labs/src/lab03/lab03_description/urdf/lab03.main.xacro (robot description, xacro)
@@ -1,74 +1,42 @@
 <?xml version="1.0"?>
 <robot xmlns:xacro="http://www.ros.org/wiki/xacro" name="lab03">
-	<!-- Include the parameters xacro flie -->
+    <!-- Include the parameters xacro flie -->
     <xacro:include filename="$(find lab03_description)/urdf/lab03.parameters.xacro" />
-    <!-- Import colors defined for Rviz -->
-    <xacro:include filename="$(find lab03_description)/urdf/lab03.rvizmats.xacro" />
     <!-- Include macros for creating all links and joints -->
     <xacro:include filename="$(find lab03_description)/urdf/lab03.macros.xacro" />
-    <!-- Add the Gazebo related elements -->
+    <!-- Include macros for creating all links and joints -->
+    <xacro:include filename="$(find lab03_description)/urdf/lab03.rvizmats.xacro" />
+    <!-- Camera in separate file for readability -->
+    <xacro:include filename="$(find lab03_description)/urdf/lab03.camera.xacro" />
+    <!-- Include gazebo elements -->
     <xacro:include filename="$(find lab03_description)/urdf/lab03.gazebo.xacro" />
-    <xacro:property name="robot_chassis_geo">
-    	<origin xyz="0 0 0" rpy="0 0 0" />
-        <geometry>
-        	<cylinder length="${ch_height}" radius="${ch_radius}"/>
-        </geometry>
-    </xacro:property>
+    <!-- Create a base link so that the robot can be away from the origin -->
     <link name="base_link" />
+    <!-- Create the robot chassis -->
     <link name="robot_chassis">
+        <!-- Create the chassis visual -->
         <visual>
-           <xacro:insert_block name="robot_chassis_geo" />
-            <material name="blue"/>
+            <xacro:create_cylinder_geometry radius="${chassis_radius}" length="${chassis_height}" />
+            <material name="white" />
         </visual>
+        <!-- The wheel's collision shape -->
         <collision>
-            <xacro:insert_block name="robot_chassis_geo" />
+            <xacro:create_cylinder_geometry radius="${chassis_radius}" length="${chassis_height}" />
         </collision>
-   		<inertial>
-            <mass value="${ch_mass}" />
-            <inertia
-                ixx="${(1/12)*ch_mass*(ch_width**2 + ch_height**2)}"
-                ixy="0"
-                ixz="0"
-                iyy="${(1/12)*ch_mass*(ch_height**2 + ch_height**2)}"
-                iyz="0"
-                izz="${(1/12)*ch_mass*(ch_height**2 + ch_width**2)}"
-                />
-        </inertial>
+        <!-- Create the chassis's inertial matrix -->
+        <xacro:create_cylinder_inertial
+            mass="${chassis_mass}" radius="${chassis_radius}"
+            length="${chassis_height}"/>
     </link>
-    <joint name="base_link_joint" type="fixed">
-        <origin xyz="0 0 ${z_offset}" rpy="0 0 0" />
+    <joint name="chassis_joint" type="fixed">
         <parent link="base_link" />
         <child link="robot_chassis" />
+        <origin xyz="0 0 ${vertical_offset}" />
     </joint>
-    <xacro:wheel reflect_lr="1" suffix="left" />s
-    <xacro:wheel reflect_lr="-1" suffix="right"/>
-    <xacro:glide reflect_lr="1" suffix="front"/>
-    <xacro:glide reflect_lr="-1" suffix="back" />
-  <!-- Camera -->
-  <link name="camera_link">
-        <visual>
-            <origin xyz="0 0 0" rpy="0 0 0"/>
-                <geometry>
-                    <box size="${camera_link} ${camera_link} ${camera_link}"/>
-                </geometry>
-                <material name="red"/>
-        </visual>
-        <collision>
-            <origin xyz="0 0 0" rpy="0 0 0"/>
-                <geometry>
-                    <box size="${camera_link} ${camera_link} ${camera_link}"/>
-                </geometry>
-        </collision>
-        <inertial>
-            <mass value="1e-5" />
-            <origin xyz="0 0 0" rpy="0 0 0"/>
-            <inertia ixx="1e-6" ixy="0" ixz="0" iyy="1e-6" iyz="0" izz="1e-6" />
-        </inertial>
-  </link>
-    <joint name="camera_joint" type="fixed">
-        <axis xyz="0 1 0" />
-        <origin xyz="0 0 ${z_offset / 2}" rpy="0 0 0" />
-        <parent link="robot_chassis"/>
-        <child link="camera_link"/>
-</joint>
+    <!-- Create the robot wheels -->
+    <xacro:create_wheel reflect_lr="1" wheel_id="left" parent_name="robot_chassis" />
+    <xacro:create_wheel reflect_lr="-1" wheel_id="right" parent_name="robot_chassis" />
+    <!-- Create the robot gliders -->
+    <xacro:create_glide reflect_fr="1" glide_id="front" parent_name="robot_chassis" />
+    <xacro:create_glide reflect_fr="-1" glide_id="rear" parent_name="robot_chassis" />
 </robot>

File: csc790_labs/src/lab03/lab03_description/urdf/lab03.parameters.xacro (robot description, xacro)
@@ -1,28 +1,33 @@
 <?xml version="1.0"?>
 <robot xmlns:xacro="http://www.ros.org/wiki/xacro" name="lab03">
-	<xacro:arg name="chassis_radius" default="0.20" />
-    <xacro:arg name="chassis_height" default="0.10" />
-    <xacro:arg name="wheel_radius" default="0.075" />
-    <xacro:arg name="glide_radius" default="0.060" />
-    <xacro:arg name="ch_width" default="0.02500" />
-    <xacro:property name="mat_density" value="1000.0" />
-    <xacro:property name="PI" value="3.1415926535897931 " />
-    <xacro:property name="SCALE" value="1.0" />
-    <xacro:property name="ch_density_factor" value="0.4" />
-    <xacro:property name="ch_density" value="${mat_density * ch_density_factor}" />
-    <xacro:property name="ch_length"  value="${0.1 * SCALE}" />
-    <xacro:property name="ch_radius"  value="$(arg chassis_radius)" />
-    <xacro:property name="ch_width"   value="${$(arg ch_width) * SCALE}" />
-    <xacro:property name="ch_height"  value="${$(arg chassis_height) * SCALE}" />
-    <xacro:property name="ch_mass"    value="${ch_density * ch_length * ch_width * ch_height}" />
-     <!-- Wheel parameters -->
-    <xacro:property name="wh_density_factor" value="0.1" />
-    <xacro:property name="wh_density" value="${mat_density * wh_density_factor}" />
-    <xacro:property name="wh_radius"  value="${$(arg wheel_radius) * SCALE}" />
-    <xacro:property name="gl_radius"  value="${$(arg glide_radius) * SCALE}" />
-    <xacro:property name="wh_length"  value="${0.005 * SCALE}" />
-    <xacro:property name="wh_mass"    value="${wh_density * PI * (wh_radius**2) * wh_length}" />
-    <xacro:property name="gl_mass"    value="${wh_density * PI * (gl_radius**2) * wh_length}" />
-    <xacro:property name="z_offset" value="${wh_radius * 2}" />
-    <xacro:property name="camera_link" value="0.05" /> <!-- Size of square 'camera' box -->
+    <!--
+         Command line arguments for the adabot
+         (See display.launch for default values)
+    -->
+    <xacro:arg name="chassis_radius" default="1" />
+    <xacro:arg name="chassis_height" default="1" />
+    <xacro:arg name="wheel_radius"   default="1" />
+    <xacro:arg name="glide_radius"   default="1" />
+    <!--
+         Properties for the robot bodies
+    -->
+    <!-- Robot vertical offset -->
+    <xacro:property name="vertical_offset" value="${wheel_radius * 1.1}" />
+    <!-- Chassis parameters -->
+    <xacro:property name="chassis_density" value="500.0" />
+    <xacro:property name="chassis_radius"  value="$(arg chassis_radius)" />
+    <xacro:property name="chassis_height"  value="$(arg chassis_height)" />
+    <xacro:property name="chassis_mass"
+        value="${chassis_density * pi * chassis_radius**2 * chassis_height}" />
+    <!-- Wheel parameters (wheel_length is only used for inertial properties)-->
+    <xacro:property name="wheel_density" value="800.0" />
+    <xacro:property name="wheel_radius"  value="$(arg wheel_radius)" />
+    <xacro:property name="wheel_length"  value="${$(arg wheel_radius) * 0.5}" />
+    <xacro:property name="wheel_mass"
+        value="${wheel_density * pi * wheel_radius**2 * wheel_length}" />
+    <!-- Glide parameters -->
+    <xacro:property name="glide_density" value="200.0" />
+    <xacro:property name="glide_radius"  value="$(arg glide_radius)" />
+    <xacro:property name="glide_mass"
+        value="${glide_density * 4.0 / 3.0 * pi * glide_radius**3}" />
 </robot>

File: csc790_labs/src/lab03/lab03_description/urdf/lab03.rvizmats.xacro (robot description, xacro)
@@ -1,12 +1,27 @@
 <?xml version="1.0"?>
 <robot xmlns:xacro="http://www.ros.org/wiki/xacro" name="lab03">
-	<material name="blue">
-    	<color rgba="0 0 0.8 1"/>
-  	</material>
-  	<material name="black">
-    	<color rgba="0 0 0 1"/>
-  	</material>
-  	<material name="white">
-    	<color rgba="1 1 1 1"/>
-  	</material>
-  </robot>
+    <material name="black">
+        <color rgba="0.0 0.0 0.0 1.0" />
+    </material>
+    <material name="blue">
+        <color rgba="0.0 0.0 0.8 1.0" />
+    </material>
+    <material name="green">
+        <color rgba="0.0 0.8 0.0 1.0" />
+    </material>
+    <material name="grey">
+        <color rgba="0.2 0.2 0.2 1.0" />
+    </material>
+    <material name="orange">
+        <color rgba="${255/255} ${108/255} ${10/255} 1.0" />
+    </material>
+    <material name="brown">
+        <color rgba="${222/255} ${207/255} ${195/255} 1.0" />
+    </material>
+    <material name="red">
+        <color rgba="0.8 0.0 0.0 1.0" />
+    </material>
+    <material name="white">
+        <color rgba="1.0 1.0 1.0 1.0" />
+    </material>
+</robot>
